File: Kicad/LED Strip clock.sch (KiCad schematic (older format))
At the start: 87 parts, among them J1 Conn_01x09_Male, J2 Conn_01x09_Male, J3 Conn_01x09_Male, J4 Conn_01x09_Male, J5 Conn_01x04_Male, J6 Barrel_Jack_Switch, U1 TPIC6B595, U10 5611BH, U11 5611BH, U12 5611BH, U13 MCP23008-xSO, U14 INA219AxD, U2 TPIC6B595, U3 TPIC6B595, U4 TPIC6B595, U5 74HCT244, U6 WeMos_D1_mini, U7 MAX809S, U8 L7805, U9 5611BH

Commit message: Change board layout. Add RTC. Add seconds LED display.
Parts:
- removed C10: 2200uF/16v, Capacitor_THT:CP_Radial_D10.0mm_P5.00mm, symbol Device:CP
- removed R39: 10K, Resistor_SMD:R_0805_2012Metric_Pad1.20x1.40mm_HandSolder, symbol Device:R
- removed TP1: TestPoint, TestPoint:TestPoint_THTPad_D1.5mm_Drill0.7mm, symbol Connector:TestPoint
- removed TP2, TP3, TP4, TP5, TP6: TestPoint, TestPoint:TestPoint_Pad_D1.0mm, symbol Connector:TestPoint
- added BT1: CR2032, Battery-extra:BatteryHolder-cr2032, symbol Device:Battery_Cell
- added C32, C33: 2200uF/16v, Capacitor_THT:CP_Radial_D10.0mm_P5.00mm, symbol Device:CP
- added C5, C6, C9: 10uF, Capacitor_SMD:C_0805_2012Metric_Pad1.18x1.45mm_HandSolder, symbol Device:C
- added D5, D6: 5611BH, Display_7Segment-extra:5611BH, symbol Display_Character-extra:5611BH
- added J5, J6: Conn_01x09_Male, Connector_PinHeader_2.54mm:PinHeader_1x09_P2.54mm_Vertical, symbol Connector:Conn_01x09_Male
- added R46, R47, R48, R49, R50, R51, R52, R53, R70, R71, R72, R73, R74, R75, R76, R77: 4K7, Resistor_SMD:R_0805_2012Metric_Pad1.20x1.40mm_HandSolder, symbol Device:R
- added U13: DS3231MZ, Package_SO:SOIC-8_3.9x4.9mm_P1.27mm, symbol Timer_RTC:DS3231MZ
- added U5, U6: TPIC6B595, Package_DIP:DIP-20_W7.62mm_LongPads, symbol Interface_Expansion-extra:TPIC6B595
- C10: renamed from C15; value 1uF -> 10uF
- C21: renamed from C12; value 33uF/16v -> 100uF/16v
- J8: renamed from J5; value Conn_01x04_Male -> Conn_01x18_Male; footprint Connector_PinHeader_2.54mm:PinHeader_1x04_P2.54mm_Vertical -> Connector_PinHeader_2.54mm:PinHeader_1x18_P2.54mm_Vertical; symbol Connector:Conn_01x04_Male -> Connector:Conn_01x18_Male
- R10: renamed from R37; value 10R -> 100R
- R11: renamed from R38; value 10R -> 100R
- R80: renamed from R40; value 10K -> 4K7
- renumbered C14 to C11, C11 to C20, C6 to C22, C7 to C23, C8 to C30, C9 to C31, C5 to C7, C13 to C8, U9 to D1, U10 to D2, U11 to D3, U12 to D4, D1 to D7, J6 to J7, R36 to R1, R1 to R12, R26 to R30, R22 to R31, R2 to R32, R6 to R33, R27 to R34, R23 to R35, R3 to R36, R7 to R37, R32 to R38, R12 to R39, R16 to R40, R20 to R41, R29 to R42, R25 to R43, R5 to R44, R9 to R45, R18 to R54, R14 to R55, R10 to R56, R30 to R57, R19 to R58, R15 to R59, R11 to R60, R31 to R61, R8 to R62, R4 to R63, R24 to R64, R28 to R65, R21 to R66, R17 to R67, R13 to R68, R33 to R69, R35 to R78, R34 to R79, U6 to U10, U13 to U11, U14 to U12, U5 to U8, U8 to U9
Connections:
- net +12V: now also J8.17 (Pin_17), C32.1, C33.1, D5.3 (CA), D5.8 (CA), D6.3 (CA), D6.8 (CA), J5.9 (Pin_9), J6.9 (Pin_9)
- net +3V3: now also J8.13 (Pin_13), C9.1, U13.2 (VCC)
- net +5V: now also J8.1 (Pin_1), J8.15 (Pin_15), C5.1, C6.1, U5.2 (VCC), U5.8 (~SRCLR), U6.2 (VCC), U6.8 (~SRCLR)
- net CLK_5V: now also U5.13 (SRCK), U6.13 (SRCK)
- net GND: now also J8.14 (Pin_14), J8.16 (Pin_16), J8.18 (Pin_18), J8.2 (Pin_2), U8.17 (2A0), BT1.2 (-), C32.2, C33.2, C5.2, C6.2, C9.2, U13.5 (GND), U5.1 (NC), U5.10 (GND), U5.11 (GND), U5.19 (GND), U5.20 (NC), U6.1 (NC), U6.10 (GND), U6.11 (GND), U6.19 (GND), U6.20 (NC); no longer J8.4 (Pin_4)
- net LATCH_5V: now also U5.12 (RCLK), U6.12 (RCLK)
- net ROT_A: now also J8.3 (Pin_3); no longer J8.1 (Pin_1)
- net ROT_B: now also J8.4 (Pin_4); no longer J8.2 (Pin_2)
- net ROT_SW: now also J8.5 (Pin_5); no longer J8.3 (Pin_3)
- net S3A: now also R40.2; no longer R63.2
- net S3B: now also R41.2; no longer R62.2
- net S3C: now also R64.2; no longer R39.2
- net S3D: now also R63.2; no longer R40.2
- net S3E: now also R62.2; no longer R41.2
- net S3F: now also R39.2; no longer R64.2
- net SCL: now also J8.11 (Pin_11), U13.8 (SCL)
- net SDA: now also J8.12 (Pin_12), U13.7 (SDA)
- net ~OE_5V: now also U5.9 (~G), U6.9 (~G)
- net ~ENBUF: now reaches U10.3 (D0)
- net ~ENBUF: now also U8.1 (1OE), U8.19 (2OE); no longer U8.17 (2A0)
- net at U4.18 (SER_OUT): now also U5.3 (SER_IN)
- net GP3: now reaches U11.13 (GP3)
- net GP3: now also J8.6 (Pin_6)
- net GP4: now reaches U11.14 (GP4)
- net GP4: now also J8.7 (Pin_7)
- net GP5: now reaches U11.15 (GP5)
- net GP5: now also J8.8 (Pin_8)
- net GP6: now reaches U11.16 (GP6)
- net GP6: now also J8.9 (Pin_9)
- net GP7: now reaches U11.17 (GP7)
- net GP7: now also J8.10 (Pin_10)
- removed net ENBUF: U10.5 (MISO/D6), U8.1 (1OE), U8.19 (2OE)
- net INT renamed INT-IO
- net VIN+: no longer names the net of F1.1, R1.2, R10.2
- new net: U5.18 (SER_OUT), U6.3 (SER_IN)
- new net: D5.5 (DP), R46.1
- new net: D5.10 (G), R73.1
- new net: D5.9 (F), R72.1
- new net: D5.1 (E), R49.1
- new net: D5.2 (D), R48.1
- new net: D5.4 (C), R47.1
- new net: D5.6 (B), R70.1
- new net: D5.7 (A), R71.1
- new net: D6.5 (DP), R77.1
- new net: D6.10 (G), R50.1
- new net: D6.9 (F), R51.1
- new net: D6.1 (E), R74.1
- new net: D6.2 (D), R75.1
- new net: D6.4 (C), R76.1
- new net: D6.6 (B), R53.1
- new net: D6.7 (A), R52.1
- new net +BATT: BT1.1 (+), U13.6 (VBAT)
- new net INT-RTC: U10.5 (MISO/D6), U13.3 (~INT~/SQW)
- new net S5A: J5.1 (Pin_1), R48.2, U5.4 (DRAIN0)
- new net S5B: J5.2 (Pin_2), R49.2, U5.5 (DRAIN1)
- new net S5C: J5.3 (Pin_3), R72.2, U5.6 (DRAIN2)
- new net S5D: J5.4 (Pin_4), R71.2, U5.7 (DRAIN3)
- new net S5DP: J5.8 (Pin_8), R46.2, U5.17 (DRAIN7)
- new net S5E: J5.5 (Pin_5), R70.2, U5.14 (DRAIN4)
- new net S5F: J5.6 (Pin_6), R47.2, U5.15 (DRAIN5)
- new net S5G: J5.7 (Pin_7), R73.2, U5.16 (DRAIN6)
- new net S6A: J6.1 (Pin_1), R52.2, U6.4 (DRAIN0)
- new net S6B: J6.2 (Pin_2), R53.2, U6.5 (DRAIN1)
- new net S6C: J6.3 (Pin_3), R76.2, U6.6 (DRAIN2)
- new net S6D: J6.4 (Pin_4), R75.2, U6.7 (DRAIN3)
- new net S6DP: J6.8 (Pin_8), R77.2, U6.17 (DRAIN7)
- new net S6E: J6.5 (Pin_5), R74.2, U6.14 (DRAIN4)
- new net S6F: J6.6 (Pin_6), R51.2, U6.15 (DRAIN5)
- new net S6G: J6.7 (Pin_7), R50.2, U6.16 (DRAIN6)
- no-connect marks 7 -> 10
Other:
- note added: "7-segment LED displays."
- note added: "CPU and I/O."
- note added: "H"
- note added: "I2C: 0x76"
- note added: "M"
- note added: "Power shift registers."
- note added: "Power supply."
- note added: "Real-time clock."
- note added: "S"
- note added: "Voltage and current measuring."
- moved on the sheet: C1, C10, C11, C2, C20, C21, C22, C23, C3, C30, C31, C4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

Commit message: Change footprint of 7805 to D2PAK.
Parts:
- U9: footprint Package_TO_SOT_SMD:TO-252-2 -> Package_TO_SOT_SMD:TO-263-2
Changed lines of the file:
@@
 Sheet 1 1
 Title "Driver for LED Strip clock"
-Date "2021-09-11"
+Date "2021-10-03"
 Rev "V1.0"
 Comp "https://github.com/atoomnetmarc/LED-Strip-clock"
@@
 F 0 "U9" H 5650 1692 50  0000 C CNN
 F 1 "L7805" H 5650 1601 50  0000 C CNN
-F 2 "Package_TO_SOT_SMD:TO-252-2" H 5675 1300 50  0001 L CIN
+F 2 "Package_TO_SOT_SMD:TO-263-2" H 5675 1300 50  0001 L CIN
 F 3 "http://www.st.com/content/ccc/resource/technical/document/datasheet/41/4f/b3/b0/12/d4/47/88/CD00000444.pdf/files/CD00000444.pdf/jcr:content/translations/en.CD00000444.pdf" H 5650 1400 50  0001 C CNN
 	1    5650 1450
