File: Kicad/LED Strip clock.kicad_pcb (KiCad board)
At the start: 2 copper layers, 142.2 x 116.8 mm, 109 parts, among them J1 Conn_01x09_Male, J2 Conn_01x09_Male, J3 Conn_01x09_Male, J4 Conn_01x09_Male, J5 Conn_01x09_Male, J6 Conn_01x09_Male, J7 Barrel_Jack_Switch, J8 Conn_01x18_Male, U1 TPIC6B595, U10 WeMos_D1_mini, U11 MCP23008-xSO, U12 INA219AxD, U13 DS3231MZ, U2 TPIC6B595, U3 TPIC6B595, U4 TPIC6B595, U5 TPIC6B595, U6 TPIC6B595, U7 MAX809S, U8 74HCT244, U9 L7805

Commit message: Add DS3231 RTC support: boot time seeding, NTP write-back and rtc CLI command
Connections:
- net /~ENBUF renamed /~{ENBUF}
- net /~OE renamed /~{OE}
- net /~OE_5V renamed /~{OE_5V}
Other:
- net class Default removed
- board text added: "16, ~{ENBUF}"
- board text added: "I2C: 0x68"
- board text added: "~{OE}, 2"
- board text removed: "16, ~ENBUF~"
- board text removed: "I2C: 0x76"
- board text removed: "~OE~, 2"
